File: mechanism-brd.brd (EAGLE design)
At the start: 100 x 80 mm, 12 parts, among them IC1 LM358N

Commit message: added platechanger.ino
Routing:
- added copper zone on layer 16, net GND
Other:
- board size 100 x 80 mm -> 61.9 x 62.2 mm
Changed lines of the file:
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@@
 <drawing>
 <settings>
-<setting alwaysvectorfont="no"/>
+<setting alwaysvectorfont="yes"/>
 <setting verticaltext="up"/>
 </settings>
@@
 <board>
 <plain>
-<wire x1="0" y1="0" x2="100" y2="0" width="0" layer="20"/>
-<wire x1="100" y1="0" x2="100" y2="80" width="0" layer="20"/>
-<wire x1="100" y1="80" x2="0" y2="80" width="0" layer="20"/>
-<wire x1="0" y1="80" x2="0" y2="0" width="0" layer="20"/>
+<wire x1="3.81" y1="2.54" x2="65.71" y2="2.54" width="0" layer="20"/>
+<wire x1="65.71" y1="2.54" x2="65.71" y2="64.76" width="0" layer="20"/>
+<wire x1="65.71" y1="64.76" x2="3.81" y2="64.76" width="0" layer="20"/>
+<wire x1="3.81" y1="64.76" x2="3.81" y2="2.54" width="0" layer="20"/>
 </plain>
 <attributes>
@@
 <wire x1="54.61" y1="39.37" x2="53.34" y2="40.64" width="1.27" layer="16"/>
 <wire x1="53.34" y1="40.64" x2="38.1" y2="40.64" width="1.27" layer="16"/>
-<wire x1="26.71" y1="27.9" x2="26.67" y2="29.21" width="0" layer="19" extent="16-16"/>
+<polygon width="0.508" layer="16" isolate="1.27">
+<vertex x="5.08" y="63.5"/>
+<vertex x="64.77" y="63.5"/>
+<vertex x="64.77" y="3.81"/>
+<vertex x="5.08" y="3.81"/>
+</polygon>
 </signal>
 <signal name="VCC">
